File: FT82_43_CMC_Choke/FT82_43_CMC_Choke.kicad_pcb (KiCad board)
At the start: 2 copper layers, 73 x 25 mm, 15 parts, among them J1 Conn_01x01_Pin, J4 Conn_01x01_Pin, J6 Conn_01x01_Pin

Commit message: Gerber for PCB v1.1
Parts:
- removed the ? at (172.5, 88.0)
- removed the ? at (180.5, 94.0)
- removed the ? at (176.5, 94.0)
- removed the ? at (172.5, 94.0)
- removed the ? at (180.5, 88.0)
- removed the ? at (176.5, 88.0)
- added ?: , , F.Cu at (188.8, 96.4)
- added ?: , , F.Cu at (190.7, 100.3)
- added ?: , , F.Cu at (184.1, 96.4)
- added ?: , , F.Cu at (179.4, 104.1)
- added ?: , , F.Cu at (184.1, 104.0)
- added ?: , , F.Cu at (179.4, 96.5)
- added ?: , , F.Cu at (188.8, 104.0)
- moved REF** 10.1 mm to (143.5, 100.2)
- moved C1 9.74 mm to (127.8, 100.2)
- moved COAX1 9.74 mm to (171.2, 102.2)
- moved F1 9.74 mm to (134.2, 102.2)
- moved F2 9.74 mm to (166.2, 98.2)
- moved J1 9.74 mm to (134.2, 98.2)
- moved J4 9.74 mm to (166.2, 102.2)
- moved J6 9.74 mm to (171.2, 98.2)
- moved REF** 9.74 mm to (150.2, 100.2)
Other:
- board size 73 x 25 mm -> 80.2 x 26.1 mm
- board text added: "(CC BY-SA 4.0)"
- board text removed: "CC BY-SA 4.0"

Commit message: PCB v1_1 :)
Other:
- board size 80.2 x 26.1 mm -> 79.6 x 26.1 mm
Changed lines of the file:
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@@
 	)
 	(gr_arc
-		(start 186.448305 91.699835)
-		(mid 194.948429 100.226401)
-		(end 186.395504 108.700001)
+		(start 186.491479 92.29992)
+		(mid 194.348343 100.249509)
+		(end 186.392462 108.100001)
 		(stroke
 			(width 0.05)
@@
 	)
 	(gr_arc
-		(start 160.210574 108.699999)
-		(mid 156.387693 111.756931)
-		(end 151.713625 113.210321)
+		(start 160.696265 108.099999)
+		(mid 156.725965 111.570978)
+		(end 151.713626 113.21032)
 		(stroke
 			(width 0.05)
@@
 	(gr_arc
 		(start 151.68258 87.159712)
-		(mid 156.373844 88.618514)
-		(end 160.2 91.700168)
+		(mid 156.710296 88.804246)
+		(end 160.680381 92.300079)
 		(stroke
 			(width 0.05)
@@
 	)
 	(gr_line
-		(start 186.395498 108.700001)
-		(end 160.210574 108.699999)
+		(start 186.392509 108.100001)
+		(end 160.696265 108.099999)
 		(stroke
 			(width 0.05)
@@
 	)
 	(gr_line
-		(start 186.448305 91.699835)
-		(end 160.2 91.7)
+		(start 186.491479 92.29992)
+		(end 160.680381 92.300079)
 		(stroke
 			(width 0.05)
