File: FT82_43_CMC_Choke/FT82_43_CMC_Choke.kicad_sch (KiCad schematic)
At the start: 7 parts, among them J1 Conn_01x01_Pin, J4 Conn_01x01_Pin, J6 Conn_01x01_Pin

Commit message: Update docs
Other:
- company: (none) -> YT3MW
- title: (none) -> QRP CMC Choke
Changed lines of the file:
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@@
 	(generator_version "9.0")
 	(paper "A4")
+	(title_block
+		(title "QRP CMC Choke")
+		(date "2026-01-02")
+		(rev "1.1")
+		(company "YT3MW")
+	)
 	(junction
 		(at 137.16 109.22)
